Commit message: S'afegeix model urdf i execució de RViz

File: urdf/IR_2.urdf (robot description, URDF)
Before this commit: robot myfirst, 1 links, 0 joints
Links:
- added link end_effector; visual sphere radius=0.08
- added link first_join; visual cylinder length=0.05 radius=0.15
- added link first_link; visual cylinder length=0.8 radius=0.06
- added link second_join; visual cylinder length=0.15 radius=0.06
- added link second_link; visual cylinder length=0.5 radius=0.06
- added link support_link; visual cylinder length=0.2 radius=0.08
- added link third_join; visual cylinder length=0.15 radius=0.06
- added link third_link; visual cylinder length=0.3 radius=0.06
- link base_link: geometry visual box size=0.6 0.6 0.2
Joints:
- added joint base_to_support: type fixed, parent base_link, child support_link, origin xyz=0 0 0.3
- added joint first_join_to_first_link: type fixed, parent first_join, child first_link, origin xyz=0 0 0.075
- added joint first_link_to_second_join: type revolute, parent first_link, child second_join, origin xyz=0 0 0.4 rpy=0 0 0, axis 0 1 0, limit lower=-2.0 upper=2.0 effort=99999 velocity=0.5
- added joint second_join_to_second_link: type fixed, parent second_join, child second_link, origin xyz=0 0 0.06
- added joint second_link_to_third_join: type revolute, parent second_link, child third_join, origin xyz=0 0 0.5 rpy=0 0 0, axis 0 1 0, limit lower=-1.0 upper=1.0 effort=99999 velocity=0.5
- added joint support_to_first_join: type continuous, parent support_link, child first_join, origin xyz=0 0 0.1, axis 0 0 1
- added joint third_join_to_third_link: type fixed, parent third_join, child third_link, origin xyz=0 0 0.06
- added joint third_link_to_end_effector: type fixed, parent third_link, child end_effector, origin xyz=0 0 0.3
